File: Hardware/PH-1200.sch (KiCad schematic (older format))
At the start: 69 parts, among them J1 SW_ONOFF, J2 SW_INV, J3 SENSOR LÍNEA, J4 RESET, J5 USB_B, J6 12V, J7 GND, K1 SRD-05VDC-SL-C, K2 SRD-05VDC-SL-C, Q1 MMBT3904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

Commit message: Update KiCad files
Parts:
- removed F2: 0.25 A, Fuse:Fuse_1206_3216Metric, symbol Device:Fuse
- removed U1: TPS562207S, Package_TO_SOT_SMD:SOT-563, symbol Regulator_Switching:TPS562207S
- added D7: B5817W, Diode_SMD:D_SOD-123, symbol Diode:B5817W
- added R22: 5.49K, Resistor_SMD:R_0603_1608Metric, symbol Device:R
- added R23: 10.2K, Resistor_SMD:R_0603_1608Metric, symbol Device:R
- added R24: 1.58K, Resistor_SMD:R_0603_1608Metric, symbol Device:R
- added U1: TPS54231DR, Package_SO:SOIC-8_3.9x4.9mm_P1.27mm, symbol Regulator_Switching:TPS54231DR
- C10: value 100nF -> 8.2nF
- C11: value 22pF -> 10pF; Voltage 16V -> 50V
- C12: value 22uF -> 6.8nF; footprint Capacitor_SMD:C_0805_2012Metric -> Capacitor_SMD:C_0402_1005Metric; Voltage 10V -> 50V
- C13: value 22uF -> 100nF; footprint Capacitor_SMD:C_0805_2012Metric -> Capacitor_SMD:C_0402_1005Metric; Dielectric (none) -> X5R or X7R
- C14: value 100nF -> 10uF; footprint Capacitor_SMD:C_0402_1005Metric -> Capacitor_SMD:C_1206_3216Metric; Voltage 10V -> 16V
- C8: value 10uF -> 22uF; footprint Capacitor_SMD:C_0805_2012Metric -> Capacitor_SMD:C_1210_3225Metric
- C9: footprint Capacitor_SMD:C_0603_1608Metric -> Capacitor_SMD:C_0402_1005Metric
- D5: footprint Diode_SMD:D_SMA -> Diode_SMD:D_SMB
- F1: value 0.5 A -> 0.75 A; Part (none) -> C1Q 750
- J6: value 12V -> GND; footprint Connector_PinHeader_2.54mm:PinHeader_1x01_P2.54mm_Vertical -> MountingHole:MountingHole_4mm_Pad
- J7: value GND -> 12V; footprint MountingHole:MountingHole_4mm_Pad -> Connector_PinHeader_2.54mm:PinHeader_1x01_P2.54mm_Vertical
- L1: value 4.7uH -> 47uH; footprint Inductor_SMD:L_Bourns_SRP7028A_7.3x6.6mm -> Inductor_SMD:L_10.4x10.4_H4.8; Part (none) -> B82464G4473M
- R20: value 64.9K -> 169K
- R21: value 10K -> 42.2K
Connections:
- wire segments 254 -> 262
Other:
- note added: "POWER SUPPLY"
- note removed: "POWER SUPPLY - 6V 0.5A"
